File: MP1/kicad/MP1.kicad_sch (KiCad schematic)
At the start: 15 parts, among them J1 USB_A, U1 MCP1702-3302E_SOT23, U2 MCP6022

Commit message: add mp1 bom
Parts:
- C1, C5: Digikey Part # (none) -> 311-1779-1-ND
- C2, C3, C4: Digikey Part # (none) -> 399-7376-1-ND
- D1: Digikey Part # (none) -> 160-1427-1-ND
- J1: Digikey Part # (none) -> WM17117-ND
- R1: Digikey Part # (none) -> 311-10.0KHRCT-ND
- R2: Digikey Part # (none) -> 311-14.3KHRCT-ND
- R3: Digikey Part # (none) -> 311-3.01MHRCT-ND
- R4: Digikey Part # (none) -> 311-9.53KHRCT-ND
- R5: Digikey Part # (none) -> 311-20.0KHRCT-ND
- R6: Digikey Part # (none) -> 311-69.8HRCT-ND
- U1: Digikey Part # (none) -> MCP1702T-3302E/CBCT-ND
- U2: Digikey Part # (none) -> MCP6022T-I/STCT-ND
Changed lines of the file:
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@@
+      (effects (font (size 1.27 1.27)) hide)
+    )
+    (property "Digikey Part #" "MCP6022T-I/STCT-ND" (id 4) (at 151.13 106.68 0)
       (effects (font (size 1.27 1.27)) hide)
     )
@@
       (effects (font (size 1.27 1.27)) hide)
     )
+    (property "Digikey Part #" "WM17117-ND" (id 4) (at 110.49 80.01 0)
+      (effects (font (size 1.27 1.27)) hide)
+    )
     (pin "1")
     (pin "2")
@@
       (effects (font (size 1.27 1.27)) hide)
     )
+    (property "Digikey Part #" "311-3.01MHRCT-ND" (id 4) (at 146.05 95.25 0)
+      (effects (font (size 1.27 1.27)) hide)
+    )
     (pin "1")
     (pin "2")
@@
       (effects (font (size 1.27 1.27)) hide)
     )
+    (property "Digikey Part #" "311-1779-1-ND" (id 4) (at 180.34 78.74 0)
+      (effects (font (size 1.27 1.27)) hide)
+    )
     (pin "1")
     (pin "2")
@@
     )
     (property "Datasheet" "http://ww1.microchip.com/downloads/en/devicedoc/20001685e.pdf" (id 3) (at 187.96 78.74 0)
+      (effects (font (size 1.27 1.27)) hide)
+    )
+    (property "Digikey Part #" "MCP6022T-I/STCT-ND" (id 4) (at 187.96 78.74 0)
       (effects (font (size 1.27 1.27)) hide)
     )
@@
       (effects (font (size 1.27 1.27)) hide)
     )
+    (property "Digikey Part #" "311-10.0KHRCT-ND" (id 4) (at 139.7 72.39 0)
+      (effects (font (size 1.27 1.27)) hide)
+    )
     (pin "1")
     (pin "2")
@@
       (effects (font (size 1.27 1.27)) hide)
     )
+    (property "Digikey Part #" "311-14.3KHRCT-ND" (id 4) (at 139.7 80.01 0)
+      (effects (font (size 1.27 1.27)) hide)
+    )
     (pin "1")
     (pin "2")
@@
       (effects (font (size 1.27 1.27)) hide)
     )
+    (property "Digikey Part #" "311-1779-1-ND" (id 4) (at 138.43 106.68 0)
+      (effects (font (size 1.27 1.27)) hide)
+    )
     (pin "1")
     (pin "2")
@@
     )
     (property "Datasheet" "~" (id 3) (at 120.65 107.95 0)
+      (effects (font (size 1.27 1.27)) hide)
+    )
+    (property "Digikey Part #" "399-7376-1-ND" (id 4) (at 120.65 107.95 0)
       (effects (font (size 1.27 1.27)) hide)
     )
@@
       (effects (font (size 1.27 1.27)) hide)
     )
+    (property "Digikey Part #" "311-69.8HRCT-ND" (id 4) (at 171.45 106.68 0)
+      (effects (font (size 1.27 1.27)) hide)
+    )
     (pin "1")
     (pin "2")
@@
       (effects (font (size 1.27 1.27)) hide)
     )
+    (property "Digikey Part #" "399-7376-1-ND" (id 4) (at 105.41 107.95 0)
+      (effects (font (size 1.27 1.27)) hide)
+    )
     (pin "1")
     (pin "2")
@@
     )
     (property "Datasheet" "~" (id 3) (at 170.18 78.74 0)
+      (effects (font (size 1.27 1.27)) hide)
+    )
+    (property "Digikey Part #" "399-7376-1-ND" (id 4) (at 170.18 78.74 0)
       (effects (font (size 1.27 1.27)) hide)
     )
@@
       (effects (font (size 1.27 1.27)) hide)
     )
+    (property "Digikey Part #" "MCP1702T-3302E/CBCT-ND" (id 4) (at 113.03 104.14 0)
+      (effects (font (size 1.27 1.27)) hide)
+    )
     (pin "1")
     (pin "2")
@@
     )
     (property "Datasheet" "~" (id 3) (at 158.75 118.11 0)
+      (effects (font (size 1.27 1.27)) hide)
+    )
+    (property "Digikey Part #" "311-20.0KHRCT-ND" (id 4) (at 158.75 118.11 0)
       (effects (font (size 1.27 1.27)) hide)
     )
@@
     )
     (property "Datasheet" "http://ww1.microchip.com/downloads/en/devicedoc/20001685e.pdf" (id 3) (at 149.86 78.74 0)
+      (effects (font (size 1.27 1.27)) hide)
+    )
+    (property "Digikey Part #" "MCP6022T-I/STCT-ND" (id 4) (at 149.86 78.74 0)
       (effects (font (size 1.27 1.27)) hide)
     )
@@
       (effects (font (size 1.27 1.27)) hide)
     )
+    (property "Digikey Part #" "311-9.53KHRCT-ND" (id 4) (at 158.75 110.49 0)
+      (effects (font (size 1.27 1.27)) hide)
+    )
     (pin "1")
     (pin "2")
@@
       (effects (font (size 1.27 1.27)) hide)
     )
+    (property "Digikey Part #" "160-1427-1-ND" (id 4) (at 179.07 106.68 0)
+      (effects (font (size 1.27 1.27)) hide)
+    )
