File: MP3/mp3.kicad_sch (KiCad schematic)
At the start: 33 parts, among them J1 USB4105-GF-A, J2 LEFT, J3 DEBUG, J4 RIGHT, U1 W25Q128JV, U2 RP2040, U3 MCP1702T-3302E_CB, Y1 12MHz

Commit message: round corners, move termination resistors close to rp2040
Connections:
- net D+: now also J1.A6 (D+), J1.B6 (D+), R6.1; no longer R6.2, U2.47 (USB_D+)
- net D-: now also J1.A7 (D-), J1.B7 (D-), R5.1; no longer R5.2, U2.46 (USB_D-)
- new net: R6.2, U2.47 (USB_D+)
- new net: R5.2, U2.46 (USB_D-)
Changed lines of the file:
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@@
     (effects (font (size 1.27 1.27)) (justify right bottom))
+  )
+  (label "D+" (at 63.5 36.83 0)
+    (effects (font (size 1.27 1.27)) (justify left bottom))
   )
   (label "GPIO17" (at 227.33 132.08 180)
@@
     (effects (font (size 1.27 1.27)) (justify right bottom))
   )
+  (label "D-" (at 68.58 31.75 0)
+    (effects (font (size 1.27 1.27)) (justify left bottom))
+  )
   (label "GPIO15" (at 194.31 134.62 0)
     (effects (font (size 1.27 1.27)) (justify left bottom))
@@
   )
   (label "GPIO12" (at 194.31 124.46 0)
-    (effects (font (size 1.27 1.27)) (justify left bottom))
-  )
-  (label "D-" (at 80.01 44.45 0)
     (effects (font (size 1.27 1.27)) (justify left bottom))
   )
@@
     (effects (font (size 1.27 1.27)) (justify left bottom))
   )
-  (label "D+" (at 80.01 49.53 0)
-    (effects (font (size 1.27 1.27)) (justify left bottom))
-  )
